Commit message: Update positions based on actual robot measurement

File: src/ros_robot_description/urdf/mecanum_robot.urdf (robot description, URDF)
Before this commit: robot mecanum_robot, 13 links, 12 joints
Joints:
- joint camera_joint: origin xyz=0.15 0 0.04 rpy=0 0 0 -> xyz=0.15 0 0.0 rpy=0 0 0
- joint laser_joint: origin xyz=0.04 0 0.11 rpy=0 0 0 -> xyz=0.12 0.0 0.09 rpy=0 0 0

Commit message: Update mecanum_robot.urdf
update to "Yaw (Z):   Rotate around vertical axis        │
│                                                                             │
│   Values in radians:                                                        │
│   • 90° = 1.5708 (π/2)                                                     │
│   • 180° = 3.14159 (π)                                                     │
│   • 270° = 4.7124 (3π/2)                                                   │
│   • 360° = 6.2832 (2π)                                                     │
│                                                                             │
│    fix: rpy="0 0 3.14159" = 180° rotation around Z  "

File: src/ros_robot_description/urdf/mecanum_robot.urdf (robot description, URDF)
Before this commit: robot mecanum_robot, 13 links, 12 joints
Joints:
- joint laser_joint: origin xyz=0.12 0.0 0.09 rpy=0 0 0 -> xyz=0.12 0.0 0.09 rpy=0 0 3.14159
